File: nano neopixel.kicad_sch (KiCad schematic)
At the start: 25 parts

Commit message: completed layout
Parts:
- added D8, D9: Conn_01x03, Connector_PinHeader_2.54mm:PinHeader_1x03_P2.54mm_Vertical, symbol Connector_Generic:Conn_01x03
- added JP7, JP8: Jumper_Open, Jumper:SolderJumper-2_P1.3mm_Open_Pad1.0x1.5mm, symbol Jumper:SolderJumper_2_Open
- added R7, R8: 470, Resistor_SMD:R_0805_2012Metric, symbol Device:R_Small_US
- C1: footprint (none) -> Capacitor_THT:CP_Radial_D8.0mm_P3.50mm; Manufactuter (none) -> Würth Elektronik; mfn (none) -> 860010274015
- renumbered Vin1 to Vin
Connections:
- net +5V: now also D8.2 (Pin_2), D9.2 (Pin_2)
- net GND: now also D8.1 (Pin_1), D9.1 (Pin_1)
- net D8: now reaches A1.11 (D8)
- net D8: now also JP7.1 (A), R7.1
- net D9: now reaches A1.12 (D9)
- net D9: now also JP8.1 (A), R8.1
- net STRIP1 renamed D2
- net STRIP2 renamed D3
- net STRIP3 renamed D4
- net STRIP4 renamed D5
- net STRIP5 renamed D6
- net STRIP6 renamed D7
- new net: D8.3 (Pin_3), JP7.2 (B), R7.2
- new net: D9.3 (Pin_3), JP8.2 (B), R8.2
- no-connect marks 0 -> 19
Other:
- company: (none) -> FRC 4488 - SHOCKWAVE
- title: (none) -> NeoPixel driver
- moved on the sheet: D2, D3, D4, D5, D6, D7, JP1, JP2, JP3, JP4, JP5, JP6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
